File: Flight_Controller_PCB/FlightController.kicad_pcb (KiCad board)
At the start: 6 copper layers, 102 x 41.1 mm, 141 parts, among them J1 TYPE-C-31-M-12, J10 Conn_01x08, J11 Conn_01x02, J12 Conn_01x08, J2 Conn_01x04_Pin, J3 Conn_01x02_Pin, J4 TYPE-C-31-M-12, J5 Conn_02x09_Top_Bottom, J6 Conn_01x08, J7 Conn_01x02, J8 Micro_SD_Card, Q1 CSD17578Q5A, Q2 CSD17578Q5A, Q3 CSD17578Q5A, Q4 CSD17578Q5A, Q5 CSD17578Q5A, Q6 Q_NPN, Q7 Q_NPN, U1 AP3211K, U10 TPS629203, U11 AMS1117-1.8, U12 TCA9534, U2 ESP32-S3-WROOM-1U-N4R8, U3 CH224K, U4 BQ25798, U5 CP2102N-Axx-xQFN28, U6 BQ7791500PWR, U7 LSM6DSOXTR, U8 MPL3115A2ST1, U9 TCA9534, Y1 ABS06-107-32.768KHZ-T

Commit message: OV5640 configuration completed, build successful
Parts:
- removed J12: Conn_01x08, TestPoint:TestPoint_THTPad_4.0x4.0mm_Drill2.0mm
- removed R41: 10k, Resistor_SMD:R_0402_1005Metric
- removed U9: TCA9534, Package_SO:TSSOP-16-1EP_4.4x5mm_P0.65mm
Connections:
- J10 pad 7: /IO14 -> /IO17
- U2 pad 11: /IO18 -> unconnected-(U2-IO18-Pad11)
- U2 pad 15: /IO3 -> /CAM_D4
- U2 pad 22: /IO14 -> /CAM_D9
- U2 pad 38: /IO2 -> /CAM_D3
- U2 pad 39: /IO1 -> /CAM_D2
- U2 pad 4: /IO4 -> /CAM_D5
- U2 pad 5: /IO5 -> /CAM_D6
- U2 pad 6: /IO6 -> /CAM_D7
- U2 pad 7: /IO7 -> /CAM_D8
Routing:
- net /IO4: track 40.0 -> 0.00 mm, vias 2 -> 0
- net /IO5: track 33.9 -> 0.00 mm, vias 1 -> 0
- net /CAM_D4: track 26.1 -> 59.9 mm, vias 0 -> 2
- net /IO6: track 32.7 -> 0.00 mm, vias 1 -> 0
- net /IO18: track 30.6 -> 0.00 mm, vias 2 -> 0
- net /IO1: track 29.5 -> 0.00 mm, vias 2 -> 0
- net /CAM_D5: track 28.5 -> 56.9 mm, vias 2 -> 3
- net /IO7: track 27.8 -> 0.00 mm, vias 2 -> 0
- net /IO3: track 23.5 -> 0.00 mm, vias 2 -> 0
- net /CAM_D6: track 18.5 -> 42.0 mm, vias 0 -> 2
- net /IO2: track 22.7 -> 0.00 mm, vias 3 -> 0
- net /CAM_D7: track 17.5 -> 39.1 mm, vias 0 -> 2
- net /CAM_D9: track 17.0 -> 37.6 mm, vias 0 -> 2
- net /CAM_D8: track 16.8 -> 36.3 mm, vias 0 -> 2
- net /IO14: track 18.0 -> 0.00 mm
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
Commit message: Added media, added STEP file of PCB
Parts:
- added R47: 10k, Resistor_SMD:R_0402_1005Metric, F.Cu at (209.9, 90.1)
- added R48: 10k, Resistor_SMD:R_0402_1005Metric, F.Cu at (209.7, 91.9)
- added R49: 10k, Resistor_SMD:R_0402_1005Metric, F.Cu at (227.0, 88.8)
- added R50: 10k, Resistor_SMD:R_0402_1005Metric, F.Cu at (221.1, 90.0)
Connections:
- J10 pad 1: /IO37 -> +3V3
- J10 pad 2: /IO36 -> /IO18
- U2 pad 11: unconnected-(U2-IO18-Pad11) -> /IO18
- U2 pad 29: /IO36 -> /PRS_INT2
- U2 pad 30: /IO37 -> /PRS_INT1
- U8 pad 5: unconnected-(U8-INT2-Pad5) -> /PRS_INT2
- U8 pad 6: unconnected-(U8-INT1-Pad6) -> /PRS_INT1
Routing:
- net /IO18: track 0.00 -> 50.6 mm, vias 0 -> 2
- net /IO37: track 35.9 -> 0.00 mm, vias 2 -> 0
- net /IO36: track 32.2 -> 0.00 mm
- net /PRS_INT2: track 0.00 -> 12.4 mm, vias 0 -> 2
- net /PRS_INT1: track 0.00 -> 11.0 mm, vias 0 -> 2
- net GND: track 69.7 -> 65.1 mm, vias 253 -> 245
- net +3V3: track 19.5 -> 21.8 mm, vias 34 -> 39
- net +1V8: track 33.1 -> 35.0 mm, vias 4 -> 5
- net /IMU_INT1: track 19.5 -> 21.2 mm, vias 2 -> 3
- net /IMU_INT2: track 18.3 -> 19.6 mm
- net /BQ_SCL: track 147.5 -> 146.7 mm
- net /IO17: track 31.2 -> 30.5 mm
- net (no net): vias 0 -> 1
Other:
- board text removed: "IO1"
- board text removed: "IO17"
- board text removed: "IO2"
- board text removed: "IO36"
- board text removed: "IO37"
- board text removed: "IO4"
- board text removed: "IO5"
- board text removed: "IO6"
- board text removed: "IO7"

Commit message: Finalize for submission and add BOM
Parts:
- removed C47: 10uF, Capacitor_SMD:C_0603_1608Metric
- removed R47, R48: 10k, Resistor_SMD:R_0402_1005Metric
- removed U8: MPL3115A2ST1, Package_LGA:NXP_LGA-8_3x5mm_P1.25mm_H1.1mm
- added U9: BME280, Package_LGA:Bosch_LGA-8_2.5x2.5mm_P0.65mm_ClockwisePinNumbering, F.Cu at (214.3, 88.2)
- L2: footprint Inductor_SMD:L_Coilcraft_XAL7020-222 -> Inductor_SMD:L_1008_2520Metric
- L3: footprint Inductor_SMD:L_Coilcraft_LPS4018 -> Inductor_SMD:L_Abracon_ASPI-4030S
- R33, R34, R35: footprint Resistor_SMD:R_0402_1005Metric -> Resistor_SMD:R_0805_2012Metric_Pad1.20x1.40mm_HandSolder; moved to B.Cu
- U10: footprint Package_SON:WSON-8-1EP_2x2mm_P0.5mm_EP0.9x1.6mm_ThermalVias -> Package_TO_SOT_SMD:SOT-583-8
- moved C46 6.44 mm to (217.3, 87.0), turned to 0 degrees
- moved C45 4.72 mm to (212.0, 88.3)
- moved L2 3.10 mm to (160.8, 75.1)
Connections:
- C45 pad 1: Net-(U8-CAP) -> +3V3
- U2 pad 29: /PRS_INT2 -> unconnected-(U2-IO36-Pad29)
- U2 pad 30: /PRS_INT1 -> unconnected-(U2-IO37-Pad30)
Routing:
- net /PRS_INT2: track 12.4 -> 0.00 mm, vias 2 -> 0
- net /PRS_INT1: track 11.0 -> 0.00 mm, vias 2 -> 0
- net /BQ_SDA: track 108.1 -> 112.5 mm
- net /TPS_VOUT: track 17.4 -> 13.4 mm
- net /BQ_SCL: track 146.7 -> 142.8 mm
- net GND: track 65.1 -> 68.7 mm, vias 245 -> 249
- net +3V3: track 21.8 -> 18.7 mm, vias 39 -> 38
- net Net-(U10-SW): track 4.60 -> 2.19 mm
- net Net-(U8-CAP): track 2.30 -> 0.00 mm
- net Net-(Q4-D): track 1.40 -> 2.80 mm, vias 0 -> 1
- net /IO18: track 50.6 -> 49.5 mm
- net /BAT_3: track 20.6 -> 20.2 mm, vias 4 -> 5
- net Net-(Q5-D): track 1.60 -> 1.84 mm, vias 0 -> 1
- net Net-(Q3-D): vias 0 -> 1
